Commit message: Removed some older versions of simple_hand, fixed up the CMakeList.txt and package.xml to make it its own package. To Do in organization: build own workspace for this project

File: simple_hand_5/urdf/simple_hand_5.urdf (robot description, URDF)
Before this commit: robot simple_hand_5, 17 links, 16 joints
Links:
- added link t1_p_r2
Joints:
- added joint thumb_palm_updown: type continuous, parent t1_p_r2, child thumb_1, origin xyz=0 0 0 rpy=0 0 0, axis 0 0 1
- joint thumb_palm: child thumb_1 -> t1_p_r2

Commit message: Added Paulina's URDF with revolute boundary conditions

File: simple_hand_5/urdf/simple_hand_5.urdf (robot description, URDF)
Before this commit: robot simple_hand_5, 18 links, 17 joints
Joints:
- joint index_12: limit (none) -> lower=0 upper=1.5708 effort=0 velocity=0; type continuous -> revolute
- joint index_23: axis 0 0 0 -> 1 0 0; limit (none) -> lower=0 upper=1.5708 effort=0 velocity=0; type fixed -> revolute
- joint index_palm: limit (none) -> lower=0 upper=1.5708 effort=0 velocity=0; type continuous -> revolute
- joint middle_12: limit lower=-1.5708 upper=0 effort=0 velocity=0 -> lower=0 upper=1.5708 effort=0 velocity=0
- joint middle_23: axis 0 0 0 -> 1 0 0; limit (none) -> lower=0 upper=1.5708 effort=0 velocity=0; type fixed -> revolute
- joint middle_palm: limit (none) -> lower=0 upper=1.5708 effort=0 velocity=0; type continuous -> revolute
- joint pinky_12: limit (none) -> lower=0 upper=1.5708 effort=0 velocity=0; type continuous -> revolute
- joint pinky_23: axis 0 0 0 -> 1 0 0; limit (none) -> lower=0 upper=1.5708 effort=0 velocity=0; type fixed -> revolute
- joint pinky_rp: limit (none) -> lower=0 upper=1.5708 effort=0 velocity=0; type continuous -> revolute
- joint ring_12: limit (none) -> lower=0 upper=1.5708 effort=0 velocity=0; type continuous -> revolute
- joint ring_23: axis 0 0 0 -> 1 0 0; limit (none) -> lower=0 upper=1.5708 effort=0 velocity=0; type fixed -> revolute
- joint ring_rp: limit (none) -> lower=0 upper=1.5708 effort=0 velocity=0; type continuous -> revolute
- joint thumb_12: limit (none) -> lower=0 upper=1.7 effort=0 velocity=0; type continuous -> revolute
- joint thumb_23: limit (none) -> lower=0 upper=1.5708 effort=0 velocity=0; type continuous -> revolute
- joint thumb_palm: limit (none) -> lower=0 upper=3.14159 effort=0 velocity=0; type continuous -> revolute
- joint thumb_palm_updown: limit (none) -> lower=-1.5708 upper=0 effort=0 velocity=0; type continuous -> revolute

Commit message: Added the rotation paths for the thumb.Paths added to hand_math.py under rot_path function.  Index and Middle touch look good, continuing to invesitgate pinky and ring. The pinky is touching but the joints are not constrained properly. Ring looks similar, but also is not at full contact point.

File: simple_hand_5/urdf/simple_hand_5.urdf (robot description, URDF)
Before this commit: robot simple_hand_5, 18 links, 17 joints
Joints:
- joint rp_palm: axis 1 0 0 -> (none); type continuous -> fixed
